Commit message: new model

File: src/robot_description/urdf/BASE_ROBOT.urdf.xacro (robot description, xacro)
@@ -1,276 +1,722 @@
 <?xml version="1.0"?>
-<robot xmlns:xacro="http://www.ros.org/wiki/xacro" name="Base">
-    <link name="dummy">
-    </link>
-    <joint name="dummy_joint" type="fixed">
-        <parent link="dummy" />
-        <child link="base_link" />
-    </joint>
-    <link name="base_link">
-        <inertial>
-            <origin
-                xyz="1.2182E-05 2.334E-05 0.0089063"
-                rpy="0 0 0" />
-            <mass
-                value=".16211" />
-            <inertia
-                ixx="0.0001472"
-                ixy="8.7863E-09"
-                ixz="-1.4391E-08"
-                iyy="0.00036976"
-                iyz="4.2045E-10"
-                izz="0.00050482" />
-        </inertial>
-        <visual>
-            <origin
-                xyz="0 0 0"
-                rpy="0 0 0" />
-            <geometry>
-                <mesh
-                    filename="package://robot_description/meshes/base_link.STL" />
-            </geometry>
-            <material
-                name="">
-                <color
-                    rgba="0.95686 0.95686 0.95686 1" />
-            </material>
-        </visual>
-        <collision>
-            <origin
-                xyz="0 0 0"
-                rpy="0 0 0" />
-            <geometry>
-                <mesh
-                    filename="package://robot_description/meshes/base_link.STL" />
-            </geometry>
-        </collision>
-    </link>
-    <link name="LBW_LINK">
-        <inertial>
-            <origin
-                xyz="5.206E-09 -4.8272E-10 -0.00089187"
-                rpy="0 0 0" />
-            <mass
-                value="0.049376" />
-            <inertia
-                ixx="1.3526E-05"
-                ixy="-6.5857E-20"
-                ixz="-5.8823E-13"
-                iyy="1.3526E-05"
-                iyz="-4.9998E-12"
-                izz="1.8891E-05" />
-        </inertial>
-        <visual>
-            <origin
-                xyz="0 0 0"
-                rpy="0 0 0" />
-            <geometry>
-                <mesh
-                    filename="package://robot_description/meshes/LBW_LINK.STL" />
-            </geometry>
-            <material
-                name="">
-                <color
-                    rgba="0.79216 0.81961 0.93333 1" />
-            </material>
-        </visual>
-        <collision>
-            <origin
-                xyz="0 0 0"
-                rpy="0 0 0" />
-            <geometry>
-                <mesh
-                    filename="package://robot_description/meshes/LBW_LINK.STL" />
-            </geometry>
-        </collision>
-    </link>
-    <joint name="LBW_JOINT" type="continuous">
-        <origin
-            xyz="-0.08315 0.075096 -0.016326"
-            rpy="-1.5708 -0.22308 0" />
-        <parent
-            link="base_link" />
-        <child
-            link="LBW_LINK" />
-        <axis
-            xyz="0 0 1" />
-        <limit
-            effort="100"
-            velocity="23.03" />
-        <dynamics
-            damping="0.1"
-            friction="0.1" />
-    </joint>
-    <link name="LFW_LINK">
-        <inertial>
-            <origin
-                xyz="5.206E-09 -4.8272E-10 -0.00089187"
-                rpy="0 0 0" />
-            <mass
-                value="0.049376" />
-            <inertia
-                ixx="1.3526E-05"
-                ixy="-7.0304E-20"
-                ixz="-5.8823E-13"
-                iyy="1.3526E-05"
-                iyz="-4.9998E-12"
-                izz="1.8891E-05" />
-        </inertial>
-        <visual>
-            <origin
-                xyz="0 0 0"
-                rpy="0 0 0" />
-            <geometry>
-                <mesh
-                    filename="package://robot_description/meshes/LFW_LINK.STL" />
-            </geometry>
-            <material
-                name="">
-                <color
-                    rgba="0.79216 0.81961 0.93333 1" />
-            </material>
-        </visual>
-        <collision>
-            <origin
-                xyz="0 0 0"
-                rpy="0 0 0" />
-            <geometry>
-                <mesh
-                    filename="package://robot_description/meshes/LFW_LINK.STL" />
-            </geometry>
-        </collision>
-    </link>
-    <joint name="LFW_JOINT"
-        type="continuous">
-        <origin
-            xyz="0.08315 0.075096 -0.016326"
-            rpy="1.5708 -1.0971 3.1416" />
-        <parent
-            link="base_link" />
-        <child
-            link="LFW_LINK" />
-        <axis
-            xyz="0 0 1" />
-        <limit
-            effort="100"
-            velocity="23.03" />
-        <dynamics
-            damping="0.1"
-            friction="0.1" />
-    </joint>
-    <link name="RBW_LINK">
-        <inertial>
-            <origin
-                xyz="5.206E-09 4.8272E-10 0.00089187"
-                rpy="0 0 0" />
-            <mass
-                value="0.049376" />
-            <inertia
-                ixx="1.3526E-05"
-                ixy="8.4756E-20"
-                ixz="5.8823E-13"
-                iyy="1.3526E-05"
-                iyz="-4.9998E-12"
-                izz="1.8891E-05" />
-        </inertial>
-        <visual>
-            <origin
-                xyz="0 0 0"
-                rpy="0 0 0" />
-            <geometry>
-                <mesh
-                    filename="package://robot_description/meshes/RBW_LINK.STL" />
-            </geometry>
-            <material
-                name="">
-                <color
-                    rgba="0.79216 0.81961 0.93333 1" />
-            </material>
-        </visual>
-        <collision>
-            <origin
-                xyz="0 0 0"
-                rpy="0 0 0" />
-            <geometry>
-                <mesh
-                    filename="package://robot_description/meshes/RBW_LINK.STL" />
-            </geometry>
-        </collision>
-    </link>
-    <joint name="RBW_JOINT"
-        type="continuous">
-        <origin
-            xyz="-0.08315 -0.075096 -0.016326"
-            rpy="1.5708 -1.5483 3.1416" />
-        <parent
-            link="base_link" />
-        <child
-            link="RBW_LINK" />
-        <axis
-            xyz="0 0 1" />
-        <limit
-            effort="100"
-            velocity="23.03" />
-        <dynamics
-            damping="0.1"
-            friction="0.1" />
-    </joint>
-    <link name="RFW_LINK">
-        <inertial>
-            <origin
-                xyz="-5.206E-09 -4.8272E-10 0.00089187"
-                rpy="0 0 0" />
-            <mass
-                value="0.049376" />
-            <inertia
-                ixx="1.3526E-05"
-                ixy="5.4634E-20"
-                ixz="-5.8823E-13"
-                iyy="1.3526E-05"
-                iyz="4.9998E-12"
-                izz="1.8891E-05" />
-        </inertial>
-        <visual>
-            <origin
-                xyz="0 0 0"
-                rpy="0 0 0" />
-            <geometry>
-                <mesh
-                    filename="package://robot_description/meshes/RFW_LINK.STL" />
-            </geometry>
-            <material
-                name="">
-                <color
-                    rgba="0.79216 0.81961 0.93333 1" />
-            </material>
-        </visual>
-        <collision>
-            <origin
-                xyz="0 0 0"
-                rpy="0 0 0" />
-            <geometry>
-                <mesh
-                    filename="package://robot_description/meshes/RFW_LINK.STL" />
-            </geometry>
-        </collision>
-    </link>
-    <joint name="RFW_JOINT"
-        type="continuous">
-        <origin
-            xyz="0.08315 -0.075096 -0.016326"
-            rpy="1.5708 -0.99328 -3.1416" />
-        <parent
-            link="base_link" />
-        <child
-            link="RFW_LINK" />
-        <axis
-            xyz="0 0 1" />
-        <limit
-            effort="100"
-            velocity="23.03" />
-        <dynamics
-            damping="0.1"
-            friction="0.1" />
-    </joint>
-<xacro:include filename="$(find robot_description)/urdf/BASE_ROBOT.gazebo"/>
+<robot xmlns:xacro="http://www.ros.org/wiki/xacro" name="Tayson">
+<xacro:include filename="$(find robot_description)/urdf/BASE_ROBOT_ESSENTIALS.xacro" />
+<xacro:include filename="$(find robot_description)/urdf/BASE_ROBOT.gazebo" />
+<material name="silver">
+  <color rgba="0.700 0.700 0.700 1.000"/>
+</material>
+<link name="dummy">
+</link>
+<joint name="dummy_joint" type="fixed">
+<parent link="dummy" />
+<child link="base_link" />
+</joint>
+<link name="base_link">
+  <inertial>
+    <origin xyz="-4.817227635489242e-16 -4.403177362975684e-17 0.044651841506048784" rpy="0 0 0"/>
+    <mass value="1.014682232407282"/>
+    <inertia ixx="0.003677" iyy="0.007865" izz="0.011516" ixy="0.0" iyz="0.0" ixz="-0.0"/>
+  </inertial>
+  <visual>
+    <origin xyz="0 0 0" rpy="0 0 0"/>
+    <geometry>
+      <mesh filename="package://robot_description/meshes/base_link.stl" scale="0.001 0.001 0.001"/>
+    </geometry>
+    <material name="silver"/>
+  </visual>
+  <collision>
+    <origin xyz="0 0 0" rpy="0 0 0"/>
+    <geometry>
+      <mesh filename="package://robot_description/meshes/base_link.stl" scale="0.001 0.001 0.001"/>
+    </geometry>
+  </collision>
+</link>
+<link name="mecanumWheelHLVR_1">
+  <inertial>
+    <origin xyz="9.020562075079397e-16 0.22810798712050598 -0.0006220000000027315" rpy="0 0 0"/>
+    <mass value="0.04937605477178852"/>
+    <inertia ixx="1.4e-05" iyy="1.9e-05" izz="1.4e-05" ixy="0.0" iyz="-0.0" ixz="0.0"/>
+  </inertial>
+  <visual>
+    <origin xyz="-0.1 0.1 -0.03145" rpy="0 0 0"/>
+    <geometry>
+      <mesh filename="package://robot_description/meshes/mecanumWheelHLVR_1.stl" scale="0.001 0.001 0.001"/>
+    </geometry>
+    <material name="silver"/>
+  </visual>
+  <collision>
+    <origin xyz="-0.1 0.1 -0.03145" rpy="0 0 0"/>
+    <geometry>
+      <mesh filename="package://robot_description/meshes/mecanumWheelHLVR_1.stl" scale="0.001 0.001 0.001"/>
+    </geometry>
+  </collision>
+</link>
+<link name="mecanumWheelHLVR_2">
+  <inertial>
+    <origin xyz="9.43689570931383e-16 0.2281079871205061 -0.000622000000004827" rpy="0 0 0"/>
+    <mass value="0.04937605477178852"/>
+    <inertia ixx="1.4e-05" iyy="1.9e-05" izz="1.4e-05" ixy="0.0" iyz="-0.0" ixz="0.0"/>
+  </inertial>
+  <visual>
+    <origin xyz="0.1 0.1 -0.03145" rpy="0 0 0"/>
+    <geometry>
+      <mesh filename="package://robot_description/meshes/mecanumWheelHLVR_2.stl" scale="0.001 0.001 0.001"/>
+    </geometry>
+    <material name="silver"/>
+  </visual>
+  <collision>
+    <origin xyz="0.1 0.1 -0.03145" rpy="0 0 0"/>
+    <geometry>
+      <mesh filename="package://robot_description/meshes/mecanumWheelHLVR_2.stl" scale="0.001 0.001 0.001"/>
+    </geometry>
+  </collision>
+</link>
+<link name="mecanumWheelHLVR_4">
+  <inertial>
+    <origin xyz="-1.4155343563970746e-15 -0.2281079871205061 -0.0006220000000028876" rpy="0 0 0"/>
+    <mass value="0.04937605477178852"/>
+    <inertia ixx="1.4e-05" iyy="1.9e-05" izz="1.4e-05" ixy="0.0" iyz="0.0" ixz="-0.0"/>
+  </inertial>
+  <visual>
+    <origin xyz="-0.1 -0.1 -0.03145" rpy="0 0 0"/>
+    <geometry>
+      <mesh filename="package://robot_description/meshes/mecanumWheelHLVR_4.stl" scale="0.001 0.001 0.001"/>
+    </geometry>
+    <material name="silver"/>
+  </visual>
+  <collision>
+    <origin xyz="-0.1 -0.1 -0.03145" rpy="0 0 0"/>
+    <geometry>
+      <mesh filename="package://robot_description/meshes/mecanumWheelHLVR_4.stl" scale="0.001 0.001 0.001"/>
+    </geometry>
+  </collision>
+</link>
+<link name="base_1">
+  <inertial>
+    <origin xyz="-0.05926053873038123 0.0008870095414633994 0.03949556593984973" rpy="0 0 0"/>
+    <mass value="0.08894964762564603"/>
+    <inertia ixx="0.000298" iyy="6.1e-05" izz="0.000351" ixy="-0.0" iyz="-0.0" ixz="-0.0"/>
+  </inertial>
+  <visual>
+    <origin xyz="-0.15 0.0 -0.014" rpy="0 0 0"/>
+    <geometry>
+      <mesh filename="package://robot_description/meshes/base_1.stl" scale="0.001 0.001 0.001"/>
+    </geometry>
+    <material name="silver"/>
+  </visual>
+  <collision>
+    <origin xyz="-0.15 0.0 -0.014" rpy="0 0 0"/>
+    <geometry>
+      <mesh filename="package://robot_description/meshes/base_1.stl" scale="0.001 0.001 0.001"/>
+    </geometry>
+  </collision>
+</link>
+<link name="Mg995_v1_1">
+  <inertial>
+    <origin xyz="-0.12433810412894816 -0.44285981612500536 -0.12727099635454053" rpy="0 0 0"/>
+    <mass value="0.029563229764879892"/>
+    <inertia ixx="4e-06" iyy="5e-06" izz="7e-06" ixy="-0.0" iyz="-0.0" ixz="0.0"/>
+  </inertial>
+  <visual>
+    <origin xyz="-0.216837 -0.37977 -0.198549" rpy="0 0 0"/>
+    <geometry>
+      <mesh filename="package://robot_description/meshes/Mg995_v1_1.stl" scale="0.001 0.001 0.001"/>
+    </geometry>
+    <material name="silver"/>
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
File: src/robot_description/urdf/BASE_ROBOT_ESSENTIALS.xacro (robot description, xacro)
@@ -1,4 +1,4 @@
 <?xml version="1.0"?>
-<robot xmlns:xacro="http://www.ros.org/wiki/xacro" name="Base">
+<robot xmlns:xacro="http://www.ros.org/wiki/xacro" name="Tayson">
 <xacro:macro name="base_transmission" params="prefix ">
 <transmission name="${prefix}_LINK_trans" type="SimpleTransmission">
@@ -13,3 +13,173 @@
 </transmission>
 </xacro:macro>
+<transmission name="hSERV_HAND_tran">
+  <type>transmission_interface/SimpleTransmission</type>
+  <joint name="hSERV_HAND">
+    <hardwareInterface>hardware_interface/EffortJointInterface</hardwareInterface>
+  </joint>
+  <actuator name="hSERV_HAND_actr">
+    <hardwareInterface>hardware_interface/EffortJointInterface</hardwareInterface>
+    <mechanicalReduction>1</mechanicalReduction>
+  </actuator>
+</transmission>
+<transmission name="BASE_FOREARM_tran">
+  <type>transmission_interface/SimpleTransmission</type>
+  <joint name="BASE_FOREARM">
+    <hardwareInterface>hardware_interface/EffortJointInterface</hardwareInterface>
+  </joint>
+  <actuator name="BASE_FOREARM_actr">
+    <hardwareInterface>hardware_interface/EffortJointInterface</hardwareInterface>
+    <mechanicalReduction>1</mechanicalReduction>
+  </actuator>
+</transmission>
+<transmission name="HAND_thumbbase_tran">
+  <type>transmission_interface/SimpleTransmission</type>
+  <joint name="HAND_thumbbase">
+    <hardwareInterface>hardware_interface/EffortJointInterface</hardwareInterface>
+  </joint>
+  <actuator name="HAND_thumbbase_actr">
+    <hardwareInterface>hardware_interface/EffortJointInterface</hardwareInterface>
+    <mechanicalReduction>1</mechanicalReduction>
+  </actuator>
+</transmission>
+<transmission name="thumbbase_thumbmiddle_tran">
+  <type>transmission_interface/SimpleTransmission</type>
+  <joint name="thumbbase_thumbmiddle">
+    <hardwareInterface>hardware_interface/EffortJointInterface</hardwareInterface>
+  </joint>
+  <actuator name="thumbbase_thumbmiddle_actr">
+    <hardwareInterface>hardware_interface/EffortJointInterface</hardwareInterface>
+    <mechanicalReduction>1</mechanicalReduction>
+  </actuator>
+</transmission>
+<transmission name="thumbmiddle_thumbtip_tran">
+  <type>transmission_interface/SimpleTransmission</type>
+  <joint name="thumbmiddle_thumbtip">
+    <hardwareInterface>hardware_interface/EffortJointInterface</hardwareInterface>
+  </joint>
+  <actuator name="thumbmiddle_thumbtip_actr">
+    <hardwareInterface>hardware_interface/EffortJointInterface</hardwareInterface>
+    <mechanicalReduction>1</mechanicalReduction>
+  </actuator>
+</transmission>
+<transmission name="HAND_pinkybase_tran">
+  <type>transmission_interface/SimpleTransmission</type>
+  <joint name="HAND_pinkybase">
+    <hardwareInterface>hardware_interface/EffortJointInterface</hardwareInterface>
+  </joint>
+  <actuator name="HAND_pinkybase_actr">
+    <hardwareInterface>hardware_interface/EffortJointInterface</hardwareInterface>
+    <mechanicalReduction>1</mechanicalReduction>
+  </actuator>
+</transmission>
+<transmission name="pinkybase_pinkymiddle_tran">
+  <type>transmission_interface/SimpleTransmission</type>
+  <joint name="pinkybase_pinkymiddle">
+    <hardwareInterface>hardware_interface/EffortJointInterface</hardwareInterface>
+  </joint>
+  <actuator name="pinkybase_pinkymiddle_actr">
+    <hardwareInterface>hardware_interface/EffortJointInterface</hardwareInterface>
+    <mechanicalReduction>1</mechanicalReduction>
+  </actuator>
+</transmission>
+<transmission name="pinkymiddle_pinkytip_tran">
+  <type>transmission_interface/SimpleTransmission</type>
+  <joint name="pinkymiddle_pinkytip">
+    <hardwareInterface>hardware_interface/EffortJointInterface</hardwareInterface>
+  </joint>
+  <actuator name="pinkymiddle_pinkytip_actr">
+    <hardwareInterface>hardware_interface/EffortJointInterface</hardwareInterface>
+    <mechanicalReduction>1</mechanicalReduction>
+  </actuator>
+</transmission>
+<transmission name="HAND_ringbase_tran">
+  <type>transmission_interface/SimpleTransmission</type>
+  <joint name="HAND_ringbase">
+    <hardwareInterface>hardware_interface/EffortJointInterface</hardwareInterface>
+  </joint>
+  <actuator name="HAND_ringbase_actr">
+    <hardwareInterface>hardware_interface/EffortJointInterface</hardwareInterface>
+    <mechanicalReduction>1</mechanicalReduction>
+  </actuator>
+</transmission>
+<transmission name="ringbase_ringmiddle_tran">
+  <type>transmission_interface/SimpleTransmission</type>
+  <joint name="ringbase_ringmiddle">
+    <hardwareInterface>hardware_interface/EffortJointInterface</hardwareInterface>
+  </joint>
+  <actuator name="ringbase_ringmiddle_actr">
+    <hardwareInterface>hardware_interface/EffortJointInterface</hardwareInterface>
+    <mechanicalReduction>1</mechanicalReduction>
+  </actuator>
+</transmission>
+<transmission name="ringmiddle_ringtip_tran">
+  <type>transmission_interface/SimpleTransmission</type>
+  <joint name="ringmiddle_ringtip">
+    <hardwareInterface>hardware_interface/EffortJointInterface</hardwareInterface>
+  </joint>
+  <actuator name="ringmiddle_ringtip_actr">
+    <hardwareInterface>hardware_interface/EffortJointInterface</hardwareInterface>
+    <mechanicalReduction>1</mechanicalReduction>
+  </actuator>
+</transmission>
+<transmission name="HAND_middlebase_tran">
+  <type>transmission_interface/SimpleTransmission</type>
+  <joint name="HAND_middlebase">
+    <hardwareInterface>hardware_interface/EffortJointInterface</hardwareInterface>
+  </joint>
+  <actuator name="HAND_middlebase_actr">
+    <hardwareInterface>hardware_interface/EffortJointInterface</hardwareInterface>
+    <mechanicalReduction>1</mechanicalReduction>
+  </actuator>
+</transmission>
+<transmission name="middlebase_middlemiddle_tran">
+  <type>transmission_interface/SimpleTransmission</type>
+  <joint name="middlebase_middlemiddle">
+    <hardwareInterface>hardware_interface/EffortJointInterface</hardwareInterface>
+  </joint>
+  <actuator name="middlebase_middlemiddle_actr">
+    <hardwareInterface>hardware_interface/EffortJointInterface</hardwareInterface>
+    <mechanicalReduction>1</mechanicalReduction>
+  </actuator>
+</transmission>
+<transmission name="middlemiddle_middletip_tran">
+  <type>transmission_interface/SimpleTransmission</type>
+  <joint name="middlemiddle_middletip">
+    <hardwareInterface>hardware_interface/EffortJointInterface</hardwareInterface>
+  </joint>
+  <actuator name="middlemiddle_middletip_actr">
+    <hardwareInterface>hardware_interface/EffortJointInterface</hardwareInterface>
+    <mechanicalReduction>1</mechanicalReduction>
+  </actuator>
+</transmission>
+<transmission name="HAND_indexbase_tran">
+  <type>transmission_interface/SimpleTransmission</type>
+  <joint name="HAND_indexbase">
+    <hardwareInterface>hardware_interface/EffortJointInterface</hardwareInterface>
+  </joint>
+  <actuator name="HAND_indexbase_actr">
+    <hardwareInterface>hardware_interface/EffortJointInterface</hardwareInterface>
+    <mechanicalReduction>1</mechanicalReduction>
+  </actuator>
+</transmission>
+<transmission name="indexbase_indexmiddle_tran">
+  <type>transmission_interface/SimpleTransmission</type>
+  <joint name="indexbase_indexmiddle">
+    <hardwareInterface>hardware_interface/EffortJointInterface</hardwareInterface>
+  </joint>
+  <actuator name="indexbase_indexmiddle_actr">
+    <hardwareInterface>hardware_interface/EffortJointInterface</hardwareInterface>
+    <mechanicalReduction>1</mechanicalReduction>
+  </actuator>
+</transmission>
+<transmission name="indexmiddle_indextip_tran">
+  <type>transmission_interface/SimpleTransmission</type>
+  <joint name="indexmiddle_indextip">
+    <hardwareInterface>hardware_interface/EffortJointInterface</hardwareInterface>
+  </joint>
+  <actuator name="indexmiddle_indextip_actr">
+    <hardwareInterface>hardware_interface/EffortJointInterface</hardwareInterface>
+    <mechanicalReduction>1</mechanicalReduction>
+  </actuator>
+</transmission>
 </robot>
