Commit message: what is happening

File: src/robot_description/urdf/BASE_ROBOT.urdf.xacro (robot description, xacro)
@@ -1,216 +1,230 @@
 <?xml version="1.0"?>
 <robot xmlns:xacro="http://www.ros.org/wiki/xacro" name="Tayson">
-<xacro:include filename="$(find robot_description)/urdf/BASE_ROBOT_ESSENTIALS.xacro" />
-<xacro:include filename="$(find robot_description)/urdf/BASE_ROBOT.gazebo" />
-<material name="silver">
-  <color rgba="0.700 0.700 0.700 1.000"/>
-</material>
-<link name="dummy">
+  <xacro:include filename="$(find robot_description)/urdf/BASE_ROBOT_ESSENTIALS.xacro" />
+  <xacro:include filename="$(find robot_description)/urdf/BASE_ROBOT.gazebo" />
+  <material name="silver">
+    <color rgba="0.700 0.700 0.700 1.000" />
+  </material>
+  <link name="dummy">
 </link>
-<joint name="dummy_joint" type="fixed">
-<parent link="dummy" />
-<child link="base_link" />
-</joint>
-<link name="base_link">
-  <inertial>
-    <origin xyz="-4.817227635489242e-16 -4.403177362975684e-17 0.044651841506048784" rpy="0 0 0"/>
-    <mass value="1.014682232407282"/>
-    <inertia ixx="0.003677" iyy="0.007865" izz="0.011516" ixy="0.0" iyz="0.0" ixz="-0.0"/>
-  </inertial>
-  <visual>
-    <origin xyz="0 0 0" rpy="0 0 0"/>
-    <geometry>
-      <mesh filename="package://robot_description/meshes/base_link.stl" scale="0.001 0.001 0.001"/>
-    </geometry>
-    <material name="silver"/>
-  </visual>
-  <collision>
-    <origin xyz="0 0 0" rpy="0 0 0"/>
-    <geometry>
-      <mesh filename="package://robot_description/meshes/base_link.stl" scale="0.001 0.001 0.001"/>
-    </geometry>
-  </collision>
-</link>
-<link name="mecanumWheelHLVR_1">
-  <inertial>
-    <origin xyz="9.020562075079397e-16 0.22810798712050598 -0.0006220000000027315" rpy="0 0 0"/>
-    <mass value="0.04937605477178852"/>
-    <inertia ixx="1.4e-05" iyy="1.9e-05" izz="1.4e-05" ixy="0.0" iyz="-0.0" ixz="0.0"/>
-  </inertial>
-  <visual>
-    <origin xyz="-0.1 0.1 -0.03145" rpy="0 0 0"/>
-    <geometry>
-      <mesh filename="package://robot_description/meshes/mecanumWheelHLVR_1.stl" scale="0.001 0.001 0.001"/>
-    </geometry>
-    <material name="silver"/>
-  </visual>
-  <collision>
-    <origin xyz="-0.1 0.1 -0.03145" rpy="0 0 0"/>
-    <geometry>
-      <mesh filename="package://robot_description/meshes/mecanumWheelHLVR_1.stl" scale="0.001 0.001 0.001"/>
-    </geometry>
-  </collision>
-</link>
-<link name="mecanumWheelHLVR_2">
-  <inertial>
-    <origin xyz="9.43689570931383e-16 0.2281079871205061 -0.000622000000004827" rpy="0 0 0"/>
-    <mass value="0.04937605477178852"/>
-    <inertia ixx="1.4e-05" iyy="1.9e-05" izz="1.4e-05" ixy="0.0" iyz="-0.0" ixz="0.0"/>
-  </inertial>
-  <visual>
-    <origin xyz="0.1 0.1 -0.03145" rpy="0 0 0"/>
-    <geometry>
-      <mesh filename="package://robot_description/meshes/mecanumWheelHLVR_2.stl" scale="0.001 0.001 0.001"/>
-    </geometry>
-    <material name="silver"/>
-  </visual>
-  <collision>
-    <origin xyz="0.1 0.1 -0.03145" rpy="0 0 0"/>
-    <geometry>
-      <mesh filename="package://robot_description/meshes/mecanumWheelHLVR_2.stl" scale="0.001 0.001 0.001"/>
-    </geometry>
-  </collision>
-</link>
-<link name="mecanumWheelHLVR_4">
-  <inertial>
-    <origin xyz="-1.4155343563970746e-15 -0.2281079871205061 -0.0006220000000028876" rpy="0 0 0"/>
-    <mass value="0.04937605477178852"/>
-    <inertia ixx="1.4e-05" iyy="1.9e-05" izz="1.4e-05" ixy="0.0" iyz="0.0" ixz="-0.0"/>
-  </inertial>
-  <visual>
-    <origin xyz="-0.1 -0.1 -0.03145" rpy="0 0 0"/>
-    <geometry>
-      <mesh filename="package://robot_description/meshes/mecanumWheelHLVR_4.stl" scale="0.001 0.001 0.001"/>
-    </geometry>
-    <material name="silver"/>
-  </visual>
-  <collision>
-    <origin xyz="-0.1 -0.1 -0.03145" rpy="0 0 0"/>
-    <geometry>
-      <mesh filename="package://robot_description/meshes/mecanumWheelHLVR_4.stl" scale="0.001 0.001 0.001"/>
-    </geometry>
-  </collision>
-</link>
-<link name="base_1">
-  <inertial>
-    <origin xyz="-0.05926053873038123 0.0008870095414633994 0.03949556593984973" rpy="0 0 0"/>
-    <mass value="0.08894964762564603"/>
-    <inertia ixx="0.000298" iyy="6.1e-05" izz="0.000351" ixy="-0.0" iyz="-0.0" ixz="-0.0"/>
-  </inertial>
-  <visual>
-    <origin xyz="-0.15 0.0 -0.014" rpy="0 0 0"/>
-    <geometry>
-      <mesh filename="package://robot_description/meshes/base_1.stl" scale="0.001 0.001 0.001"/>
-    </geometry>
-    <material name="silver"/>
-  </visual>
-  <collision>
-    <origin xyz="-0.15 0.0 -0.014" rpy="0 0 0"/>
-    <geometry>
-      <mesh filename="package://robot_description/meshes/base_1.stl" scale="0.001 0.001 0.001"/>
-    </geometry>
-  </collision>
-</link>
-<link name="Mg995_v1_1">
-  <inertial>
-    <origin xyz="-0.12433810412894816 -0.44285981612500536 -0.12727099635454053" rpy="0 0 0"/>
-    <mass value="0.029563229764879892"/>
-    <inertia ixx="4e-06" iyy="5e-06" izz="7e-06" ixy="-0.0" iyz="-0.0" ixz="0.0"/>
-  </inertial>
-  <visual>
-    <origin xyz="-0.216837 -0.37977 -0.198549" rpy="0 0 0"/>
-    <geometry>
-      <mesh filename="package://robot_description/meshes/Mg995_v1_1.stl" scale="0.001 0.001 0.001"/>
-    </geometry>
-    <material name="silver"/>
-  </visual>
-  <collision>
-    <origin xyz="-0.216837 -0.37977 -0.198549" rpy="0 0 0"/>
-    <geometry>
-      <mesh filename="package://robot_description/meshes/Mg995_v1_1.stl" scale="0.001 0.001 0.001"/>
-    </geometry>
-  </collision>
-</link>
-<link name="Mg995_v1__2__1">
-  <inertial>
-    <origin xyz="-0.12433810412894808 -0.45162532874216155 -0.1272710036454569" rpy="0 0 0"/>
-    <mass value="0.029563229764879892"/>
-    <inertia ixx="4e-06" iyy="5e-06" izz="7e-06" ixy="0.0" iyz="-0.0" ixz="-0.0"/>
-  </inertial>
-  <visual>
-    <origin xyz="-0.216837 -0.519507 -0.198549" rpy="0 0 0"/>
-    <geometry>
-      <mesh filename="package://robot_description/meshes/Mg995_v1__2__1.stl" scale="0.001 0.001 0.001"/>
-    </geometry>
-    <material name="silver"/>
-  </visual>
-  <collision>
-    <origin xyz="-0.216837 -0.519507 -0.198549" rpy="0 0 0"/>
-    <geometry>
-      <mesh filename="package://robot_description/meshes/Mg995_v1__2__1.stl" scale="0.001 0.001 0.001"/>
-    </geometry>
-  </collision>
-</link>
-<link name="Mg995_v1__1__1">
-  <inertial>
-    <origin xyz="-0.13683854098619236 -0.009229321224777876 -0.5693955665007882" rpy="0 0 0"/>
-    <mass value="0.029563229764879892"/>
-    <inertia ixx="7e-06" iyy="4e-06" izz="5e-06" ixy="0.0" iyz="-0.0" ixz="-0.0"/>
-  </inertial>
-  <visual>
-    <origin xyz="-0.0975233 -0.005736 -0.273127" rpy="0 0 0"/>
-    <geometry>
-      <mesh filename="package://robot_description/meshes/Mg995_v1__1__1.stl" scale="0.001 0.001 0.001"/>
-    </geometry>
-    <material name="silver"/>
-  </visual>
-  <collision>
-    <origin xyz="-0.0975233 -0.005736 -0.273127" rpy="0 0 0"/>
-    <geometry>
-      <mesh filename="package://robot_description/meshes/Mg995_v1__1__1.stl" scale="0.001 0.001 0.001"/>
-    </geometry>
-  </collision>
-</link>
-<link name="HAND_BASE_PROTO_VER_2_1">
-  <inertial>
-    <origin xyz="-0.2727629292240147 -0.0962305740932451 0.08548535560636134" rpy="0 0 0"/>
-    <mass value="0.1827874583391763"/>
-    <inertia ixx="0.000592" iyy="0.000397" izz="0.000225" ixy="1.7e-05" iyz="-5.5e-05" ixz="1.9e-05"/>
-  </inertial>
-  <visual>
-    <origin xyz="-0.1005902 -0.0202162 -0.2962644" rpy="0 0 0"/>
-    <geometry>
-      <mesh filename="package://robot_description/meshes/HAND_BASE_PROTO_VER_2_1.stl" scale="0.001 0.001 0.001"/>
-    </geometry>
-    <material name="silver"/>
-  </visual>
-  <collision>
-    <origin xyz="-0.1005902 -0.0202162 -0.2962644" rpy="0 0 0"/>
-    <geometry>
-      <mesh filename="package://robot_description/meshes/HAND_BASE_PROTO_VER_2_1.stl" scale="0.001 0.001 0.001"/>
-    </geometry>
-  </collision>
-</link>
-<link name="forearm_1">
-  <inertial>
-    <origin xyz="0.009963523872911717 -0.00039503291108781025 0.11306234197836312" rpy="0 0 0"/>
-    <mass value="0.16311330061478566"/>
-    <inertia ixx="0.000769" iyy="0.00065" izz="0.000138" ixy="-0.0" iyz="1e-06" ixz="-0.0"/>
-  </inertial>
-  <visual>
-    <origin xyz="-0.102233 -0.002396 -0.061278" rpy="0 0 0"/>
-    <geometry>
-      <mesh filename="package://robot_description/meshes/forearm_1.stl" scale="0.001 0.001 0.001"/>
-    </geometry>
-    <material name="silver"/>
-  </visual>
-  <collision>
-    <origin xyz="-0.102233 -0.002396 -0.061278" rpy="0 0 0"/>
-    <geometry>
-      <mesh filename="package://robot_description/meshes/forearm_1.stl" scale="0.001 0.001 0.001"/>
-    </geometry>
-  </collision>
-</link>
-<!--<link name="pinky_finger_base_2">
+  <joint name="dummy_joint" type="fixed">
+    <parent link="dummy" />
+    <child link="base_link" />
+  </joint>
+  <link name="base_link">
+    <inertial>
+      <origin xyz="-4.817227635489242e-16 -4.403177362975684e-17 0.044651841506048784" rpy="0 0 0" />
+      <mass value="100.014682232407282" />
+      <inertia ixx="0.003677" iyy="0.007865" izz="0.011516" ixy="0.0" iyz="0.0" ixz="-0.0" />
+    </inertial>
+    <visual>
+      <origin xyz="0 0 0" rpy="0 0 0" />
+      <geometry>
+        <mesh filename="package://robot_description/meshes/base_link.stl" scale="0.001 0.001 0.001" />
+      </geometry>
+      <material name="silver" />
+    </visual>
+    <collision>
+      <origin xyz="0 0 0" rpy="0 0 0" />
+      <geometry>
+        <mesh filename="package://robot_description/meshes/base_link.stl" scale="0.001 0.001 0.001" />
+      </geometry>
+    </collision>
+  </link>
+  <link name="mecanumWheelHLVR_1">
+    <inertial>
+      <origin xyz="9.020562075079397e-16 0.22810798712050598 -0.0006220000000027315" rpy="0 0 0" />
+      <mass value="0.04937605477178852" />
+      <inertia ixx="1.4e-05" iyy="1.9e-05" izz="1.4e-05" ixy="0.0" iyz="-0.0" ixz="0.0" />
+    </inertial>
+    <visual>
+      <origin xyz="-0.1 0.1 -0.03145" rpy="0 0 0" />
+      <geometry>
+        <mesh filename="package://robot_description/meshes/mecanumWheelHLVR_1.stl"
+          scale="0.001 0.001 0.001" />
+      </geometry>
+      <material name="silver" />
+    </visual>
+    <collision>
+      <origin xyz="-0.1 0.1 -0.03145" rpy="0 0 0" />
+      <geometry>
+        <mesh filename="package://robot_description/meshes/mecanumWheelHLVR_1.stl"
+          scale="0.001 0.001 0.001" />
+      </geometry>
+    </collision>
+  </link>
+  <link name="mecanumWheelHLVR_2">
+    <inertial>
+      <origin xyz="9.43689570931383e-16 0.2281079871205061 -0.000622000000004827" rpy="0 0 0" />
+      <mass value="0.04937605477178852" />
+      <inertia ixx="1.4e-05" iyy="1.9e-05" izz="1.4e-05" ixy="0.0" iyz="-0.0" ixz="0.0" />
+    </inertial>
+    <visual>
+      <origin xyz="0.1 0.1 -0.03145" rpy="0 0 0" />
+      <geometry>
+        <mesh filename="package://robot_description/meshes/mecanumWheelHLVR_2.stl"
+          scale="0.001 0.001 0.001" />
+      </geometry>
+      <material name="silver" />
+    </visual>
+    <collision>
+      <origin xyz="0.1 0.1 -0.03145" rpy="0 0 0" />
+      <geometry>
+        <mesh filename="package://robot_description/meshes/mecanumWheelHLVR_2.stl"
+          scale="0.001 0.001 0.001" />
+      </geometry>
+    </collision>
+  </link>
+  <link name="mecanumWheelHLVR_4">
+    <inertial>
+      <origin xyz="-1.4155343563970746e-15 -0.2281079871205061 -0.0006220000000028876" rpy="0 0 0" />
+      <mass value="0.04937605477178852" />
+      <inertia ixx="1.4e-05" iyy="1.9e-05" izz="1.4e-05" ixy="0.0" iyz="0.0" ixz="-0.0" />
+    </inertial>
+    <visual>
+      <origin xyz="-0.1 -0.1 -0.03145" rpy="0 0 0" />
+      <geometry>
+        <mesh filename="package://robot_description/meshes/mecanumWheelHLVR_4.stl"
+          scale="0.001 0.001 0.001" />
+      </geometry>
+      <material name="silver" />
+    </visual>
+    <collision>
+      <origin xyz="-0.1 -0.1 -0.03145" rpy="0 0 0" />
+      <geometry>
+        <mesh filename="package://robot_description/meshes/mecanumWheelHLVR_4.stl"
+          scale="0.001 0.001 0.001" />
+      </geometry>
+    </collision>
+  </link>
+  <link name="base_1">
+    <inertial>
+      <origin xyz="-0.05926053873038123 0.0008870095414633994 0.03949556593984973" rpy="0 0 0" />
+      <mass value="0.08894964762564603" />
+      <inertia ixx="0.000298" iyy="6.1e-05" izz="0.000351" ixy="-0.0" iyz="-0.0" ixz="-0.0" />
+    </inertial>
+    <visual>
+      <origin xyz="-0.15 0.0 -0.014" rpy="0 0 0" />
+      <geometry>
+        <mesh filename="package://robot_description/meshes/base_1.stl" scale="0.001 0.001 0.001" />
+      </geometry>
+      <material name="silver" />
+    </visual>
+    <collision>
+      <origin xyz="-0.15 0.0 -0.014" rpy="0 0 0" />
+      <geometry>
+        <mesh filename="package://robot_description/meshes/base_1.stl" scale="0.001 0.001 0.001" />
+      </geometry>
+    </collision>
+  </link>
+  <link name="Mg995_v1_1">
+    <inertial>
+      <origin xyz="-0.12433810412894816 -0.44285981612500536 -0.12727099635454053" rpy="0 0 0" />
+      <mass value="0.029563229764879892" />
+      <inertia ixx="4e-06" iyy="5e-06" izz="7e-06" ixy="-0.0" iyz="-0.0" ixz="0.0" />
+    </inertial>
+    <visual>
+      <origin xyz="-0.216837 -0.37977 -0.198549" rpy="0 0 0" />
+      <geometry>
+        <mesh filename="package://robot_description/meshes/Mg995_v1_1.stl" scale="0.001 0.001 0.001" />
+      </geometry>
+      <material name="silver" />
+    </visual>
+    <collision>
+      <origin xyz="-0.216837 -0.37977 -0.198549" rpy="0 0 0" />
+      <geometry>
+        <mesh filename="package://robot_description/meshes/Mg995_v1_1.stl" scale="0.001 0.001 0.001" />
+      </geometry>
+    </collision>
+  </link>
+  <link name="Mg995_v1__2__1">
+    <inertial>
+      <origin xyz="-0.12433810412894808 -0.45162532874216155 -0.1272710036454569" rpy="0 0 0" />
+      <mass value="0.029563229764879892" />
+      <inertia ixx="4e-06" iyy="5e-06" izz="7e-06" ixy="0.0" iyz="-0.0" ixz="-0.0" />
+    </inertial>
+    <visual>
+      <origin xyz="-0.216837 -0.519507 -0.198549" rpy="0 0 0" />
+      <geometry>
+        <mesh filename="package://robot_description/meshes/Mg995_v1__2__1.stl"
+          scale="0.001 0.001 0.001" />
+      </geometry>
+      <material name="silver" />
+    </visual>
+    <collision>
+      <origin xyz="-0.216837 -0.519507 -0.198549" rpy="0 0 0" />
+      <geometry>
+        <mesh filename="package://robot_description/meshes/Mg995_v1__2__1.stl"
+          scale="0.001 0.001 0.001" />
+      </geometry>
+    </collision>
+  </link>
+  <link name="Mg995_v1__1__1">
+    <inertial>
+      <origin xyz="-0.13683854098619236 -0.009229321224777876 -0.5693955665007882" rpy="0 0 0" />
+      <mass value="0.029563229764879892" />
+      <inertia ixx="7e-06" iyy="4e-06" izz="5e-06" ixy="0.0" iyz="-0.0" ixz="-0.0" />
+    </inertial>
+    <visual>
+      <origin xyz="-0.0975233 -0.005736 -0.273127" rpy="0 0 0" />
+      <geometry>
+        <mesh filename="package://robot_description/meshes/Mg995_v1__1__1.stl"
+          scale="0.001 0.001 0.001" />
+      </geometry>
+      <material name="silver" />
+    </visual>
+    <collision>
+      <origin xyz="-0.0975233 -0.005736 -0.273127" rpy="0 0 0" />
+      <geometry>
+        <mesh filename="package://robot_description/meshes/Mg995_v1__1__1.stl"
+          scale="0.001 0.001 0.001" />
+      </geometry>
+    </collision>
+  </link>
+  <link name="HAND_BASE_PROTO_VER_2_1">
+    <inertial>
+      <origin xyz="-0.2727629292240147 -0.0962305740932451 0.08548535560636134" rpy="0 0 0" />
+      <mass value="0.1827874583391763" />
+      <inertia ixx="0.000592" iyy="0.000397" izz="0.000225" ixy="1.7e-05" iyz="-5.5e-05"
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