Commit message: effort controllers working

File: src/robot_description/urdf/BASE_ROBOT.urdf.xacro (robot description, xacro)
@@ -7,5 +7,5 @@
   </material>
   <link name="dummy">
-</link>
+  </link>
   <joint name="dummy_joint" type="fixed">
     <parent link="dummy" />
@@ -15,5 +15,5 @@
     <inertial>
       <origin xyz="-4.817227635489242e-16 -4.403177362975684e-17 0.044651841506048784" rpy="0 0 0" />
-      <mass value="100.014682232407282" />
+      <mass value="10.014682232407282" />
       <inertia ixx="0.003677" iyy="0.007865" izz="0.011516" ixy="0.0" iyz="0.0" ixz="-0.0" />
     </inertial>
@@ -98,4 +98,26 @@
     </collision>
   </link>
+  <link name="mecanumWheelHLVR_3">
+    <inertial>
+      <origin xyz="-3.885780586188048e-15 -0.2271079871205061 -0.0006220000000000288" rpy="0 0 0" />
+      <mass value="0.04937605477178852" />
+      <inertia ixx="1.4e-05" iyy="1.9e-05" izz="1.4e-05" ixy="0.0" iyz="-0.0" ixz="0.0" />
+    </inertial>
+    <visual>
+      <origin xyz="0.1 -0.1 -0.03145" rpy="0 0 0" />
+      <geometry>
+        <mesh filename="package://robot_description/meshes/mecanumWheelHLVR_3.stl"
+          scale="0.001 0.001 0.001" />
+      </geometry>
+      <material name="silver" />
+    </visual>
+    <collision>
+      <origin xyz="0.1 -0.1 -0.03145" rpy="0 0 0" />
+      <geometry>
+        <mesh filename="package://robot_description/meshes/mecanumWheelHLVR_3.stl"
+          scale="0.001 0.001 0.001" />
+      </geometry>
+    </collision>
+  </link>
   <link name="base_1">
     <inertial>
@@ -157,4 +179,24 @@
         <mesh filename="package://robot_description/meshes/Mg995_v1__2__1.stl"
           scale="0.001 0.001 0.001" />
+      </geometry>
+    </collision>
+  </link>
+  <link name="forearm_1">
+    <inertial>
+      <origin xyz="0.009963523872911717 -0.00039503291108781025 0.11306234197836312" rpy="0 0 0" />
+      <mass value="0.16311330061478566" />
+      <inertia ixx="0.000769" iyy="0.00065" izz="0.000138" ixy="-0.0" iyz="1e-06" ixz="-0.0" />
+    </inertial>
+    <visual>
+      <origin xyz="-0.102233 -0.002396 -0.061278" rpy="0 0 0" />
+      <geometry>
+        <mesh filename="package://robot_description/meshes/forearm_1.stl" scale="0.001 0.001 0.001" />
+      </geometry>
+      <material name="silver" />
+    </visual>
+    <collision>
+      <origin xyz="-0.102233 -0.002396 -0.061278" rpy="0 0 0" />
+      <geometry>
+        <mesh filename="package://robot_description/meshes/forearm_1.stl" scale="0.001 0.001 0.001" />
       </geometry>
     </collision>
@@ -205,91 +247,99 @@
     </collision>
   </link>
-  <link name="forearm_1">
-    <inertial>
-      <origin xyz="0.009963523872911717 -0.00039503291108781025 0.11306234197836312" rpy="0 0 0" />
-      <mass value="0.16311330061478566" />
-      <inertia ixx="0.000769" iyy="0.00065" izz="0.000138" ixy="-0.0" iyz="1e-06" ixz="-0.0" />
-    </inertial>
-    <visual>
-      <origin xyz="-0.102233 -0.002396 -0.061278" rpy="0 0 0" />
-      <geometry>
-        <mesh filename="package://robot_description/meshes/forearm_1.stl" scale="0.001 0.001 0.001" />
-      </geometry>
-      <material name="silver" />
-    </visual>
-    <collision>
-      <origin xyz="-0.102233 -0.002396 -0.061278" rpy="0 0 0" />
-      <geometry>
-        <mesh filename="package://robot_description/meshes/forearm_1.stl" scale="0.001 0.001 0.001" />
-      </geometry>
-    </collision>
-  </link>
-  <!--<link
-  name="pinky_finger_base_2">
-  <inertial>
-    <origin xyz="0.12562978099685648 -0.439944340852892 -0.2543173869988929" rpy="0 0 0"/>
-    <mass value="0.01136811456417231"/>
-    <inertia ixx="2e-06" iyy="3e-06" izz="2e-06" ixy="-0.0" iyz="-0.0" ixz="-1e-06"/>
-  </inertial>
-  <visual>
-    <origin xyz="-0.019849 -0.384881 -0.642689" rpy="0 0 0"/>
-    <geometry>
-      <mesh filename="package://robot_description/meshes/pinky_finger_base_2.stl" scale="0.001 0.001
-  0.001"/>
-    </geometry>
-    <material name="silver"/>
-  </visual>
-  <collision>
-    <origin xyz="-0.019849 -0.384881 -0.642689" rpy="0 0 0"/>
-    <geometry>
-      <mesh filename="package://robot_description/meshes/pinky_finger_base_2.stl" scale="0.001 0.001
-  0.001"/>
-    </geometry>
-  </collision>
-</link>
-<link name="pinky_finger_middle_2">
-  <inertial>
-    <origin xyz="0.0816570642888089 -0.12487104495808517 -0.06840307826125513" rpy="0 0 0"/>
-    <mass value="0.006674601249639396"/>
-    <inertia ixx="1e-06" iyy="1e-06" izz="1e-06" ixy="-0.0" iyz="-0.0" ixz="-0.0"/>
-  </inertial>
-  <visual>
-    <origin xyz="-0.095583 -0.073585 -0.487214" rpy="0 0 0"/>
-    <geometry>
-      <mesh filename="package://robot_description/meshes/pinky_finger_middle_2.stl" scale="0.001 0.001
-  0.001"/>
-    </geometry>
-    <material name="silver"/>
-  </visual>
-  <collision>
-    <origin xyz="-0.095583 -0.073585 -0.487214" rpy="0 0 0"/>
-    <geometry>
-      <mesh filename="package://robot_description/meshes/pinky_finger_middle_2.stl" scale="0.001 0.001
-  0.001"/>
-    </geometry>
-  </collision>
-</link>
-<link name="pinky_finger_tip_2">
-  <inertial>
-    <origin xyz="0.10624000517014226 -0.11513256790913157 -0.07884189536515152" rpy="0 0 0"/>
-    <mass value="0.0045834007133138035"/>
-    <inertia ixx="0.0" iyy="1e-06" izz="0.0" ixy="-0.0" iyz="-0.0" ixz="-0.0"/>
-  </inertial>
-  <visual>
-    <origin xyz="-0.095696 -0.067585 -0.521214" rpy="0 0 0"/>
-    <geometry>
-      <mesh filename="package://robot_description/meshes/pinky_finger_tip_2.stl" scale="0.001 0.001
-  0.001"/>
-    </geometry>
-    <material name="silver"/>
-  </visual>
-  <collision>
-    <origin xyz="-0.095696 -0.067585 -0.521214" rpy="0 0 0"/>
-    <geometry>
-      <mesh filename="package://robot_description/meshes/pinky_finger_tip_2.stl" scale="0.001 0.001
-  0.001"/>
-    </geometry>
-  </collision>
-</link>-->
+  <link name="TOP_COVER_PROTO_VER2_1">
+    <inertial>
+      <origin xyz="-0.022679449260790477 0.053604413909800544 -0.01649356765285831" rpy="0 0 0" />
+      <mass value="0.0491327525476126" />
+      <inertia ixx="0.000183" iyy="8.7e-05" izz="0.000121" ixy="8e-06" iyz="-2e-06" ixz="9e-06" />
+    </inertial>
+    <visual>
+      <origin xyz="-0.103733 0.044258 -0.381814" rpy="0 0 0" />
+      <geometry>
+        <mesh filename="package://robot_description/meshes/TOP_COVER_PROTO_VER2_1.stl"
+          scale="0.001 0.001 0.001" />
+      </geometry>
+      <material name="silver" />
+    </visual>
+    <collision>
+      <origin xyz="-0.103733 0.044258 -0.381814" rpy="0 0 0" />
+      <geometry>
+        <mesh filename="package://robot_description/meshes/TOP_COVER_PROTO_VER2_1.stl"
+          scale="0.001 0.001 0.001" />
+      </geometry>
+    </collision>
+  </link>
+  <!-- <link
+    name="pinky_finger_base_2">
+    <inertial>
+      <origin xyz="0.12562978099685648 -0.439944340852892 -0.2543173869988929" rpy="0 0 0" />
+      <mass value="0.01136811456417231" />
+      <inertia ixx="2e-06" iyy="3e-06" izz="2e-06" ixy="-0.0" iyz="-0.0" ixz="-1e-06" />
+    </inertial>
+    <visual>
+      <origin xyz="-0.019849 -0.384881 -0.642689" rpy="0 0 0" />
+      <geometry>
+        <mesh filename="package://robot_description/meshes/pinky_finger_base_2.stl"
+          scale="0.001 0.001
+  0.001" />
+      </geometry>
+      <material name="silver" />
+    </visual>
+    <collision>
+      <origin xyz="-0.019849 -0.384881 -0.642689" rpy="0 0 0" />
+      <geometry>
+        <mesh filename="package://robot_description/meshes/pinky_finger_base_2.stl"
+          scale="0.001 0.001
+  0.001" />
+      </geometry>
+    </collision>
+  </link>
+  <link name="pinky_finger_middle_2">
+    <inertial>
+      <origin xyz="0.0816570642888089 -0.12487104495808517 -0.06840307826125513" rpy="0 0 0" />
+      <mass value="0.006674601249639396" />
+      <inertia ixx="1e-06" iyy="1e-06" izz="1e-06" ixy="-0.0" iyz="-0.0" ixz="-0.0" />
+    </inertial>
+    <visual>
+      <origin xyz="-0.095583 -0.073585 -0.487214" rpy="0 0 0" />
+      <geometry>
+        <mesh filename="package://robot_description/meshes/pinky_finger_middle_2.stl"
+          scale="0.001 0.001
+  0.001" />
+      </geometry>
+      <material name="silver" />
+    </visual>
+    <collision>
+      <origin xyz="-0.095583 -0.073585 -0.487214" rpy="0 0 0" />
+      <geometry>
+        <mesh filename="package://robot_description/meshes/pinky_finger_middle_2.stl"
+          scale="0.001 0.001
+  0.001" />
+      </geometry>
+    </collision>
+  </link>
+  <link name="pinky_finger_tip_2">
+    <inertial>
+      <origin xyz="0.10624000517014226 -0.11513256790913157 -0.07884189536515152" rpy="0 0 0" />
+      <mass value="0.0045834007133138035" />
+      <inertia ixx="0.0" iyy="1e-06" izz="0.0" ixy="-0.0" iyz="-0.0" ixz="-0.0" />
+    </inertial>
+    <visual>
+      <origin xyz="-0.095696 -0.067585 -0.521214" rpy="0 0 0" />
+      <geometry>
+        <mesh filename="package://robot_description/meshes/pinky_finger_tip_2.stl"
+          scale="0.001 0.001
+  0.001" />
+      </geometry>
+      <material name="silver" />
+    </visual>
+    <collision>
+      <origin xyz="-0.095696 -0.067585 -0.521214" rpy="0 0 0" />
+      <geometry>
+        <mesh filename="package://robot_description/meshes/pinky_finger_tip_2.stl"
+          scale="0.001 0.001
+  0.001" />
+      </geometry>
+    </collision>
+  </link> -->
   <link name="pinky_finger_base_1">
     <inertial>
@@ -552,48 +602,4 @@
       <geometry>
         <mesh filename="package://robot_description/meshes/index_finger_tip_2.stl"
-          scale="0.001 0.001 0.001" />
-      </geometry>
-    </collision>
-  </link>
-  <link name="TOP_COVER_PROTO_VER2_1">
-    <inertial>
-      <origin xyz="-0.022679449260790477 0.053604413909800544 -0.01649356765285831" rpy="0 0 0" />
-      <mass value="0.0491327525476126" />
-      <inertia ixx="0.000183" iyy="8.7e-05" izz="0.000121" ixy="8e-06" iyz="-2e-06" ixz="9e-06" />
-    </inertial>
-    <visual>
-      <origin xyz="-0.103733 0.044258 -0.381814" rpy="0 0 0" />
-      <geometry>
-        <mesh filename="package://robot_description/meshes/TOP_COVER_PROTO_VER2_1.stl"
-          scale="0.001 0.001 0.001" />
-      </geometry>
-      <material name="silver" />
-    </visual>
-    <collision>
-      <origin xyz="-0.103733 0.044258 -0.381814" rpy="0 0 0" />
-      <geometry>
-        <mesh filename="package://robot_description/meshes/TOP_COVER_PROTO_VER2_1.stl"
-          scale="0.001 0.001 0.001" />
-      </geometry>
-    </collision>
-  </link>
-  <link name="mecanumWheelHLVR_3">
-    <inertial>
-      <origin xyz="-3.885780586188048e-15 -0.2271079871205061 -0.0006220000000000288" rpy="0 0 0" />
-      <mass value="0.04937605477178852" />
-      <inertia ixx="1.4e-05" iyy="1.9e-05" izz="1.4e-05" ixy="0.0" iyz="-0.0" ixz="0.0" />
-    </inertial>
-    <visual>
-      <origin xyz="0.1 -0.1 -0.03145" rpy="0 0 0" />
-      <geometry>
-        <mesh filename="package://robot_description/meshes/mecanumWheelHLVR_3.stl"
-          scale="0.001 0.001 0.001" />
-      </geometry>
-      <material name="silver" />
-    </visual>
-    <collision>
-      <origin xyz="0.1 -0.1 -0.03145" rpy="0 0 0" />
-      <geometry>
-        <mesh filename="package://robot_description/meshes/mecanumWheelHLVR_3.stl"
           scale="0.001 0.001 0.001" />
       </geometry>
@@ -638,4 +644,11 @@
     <parent link="base_1" />
     <child link="Mg995_v1__2__1" />
+  </joint>
+  <joint name="BASE_FOREARM" type="revolute">
+    <origin xyz="-0.048667 0.002396 0.047278" rpy="0 0 0" />
+    <parent link="base_1" />
+    <child link="forearm_1" />
+    <axis xyz="-0.0 -1.0 -0.0" />
+    <limit upper="1.57" lower="-1.57" effort="50" velocity="-1" />
   </joint>
   <joint name="FOREARM_hSERV" type="fixed">
@@ -651,12 +664,79 @@
     <limit upper="1.570796" lower="-1.57" effort="100" velocity="100" />
   </joint>
-  <joint name="BASE_FOREARM" type="revolute">
-    <origin xyz="-0.048667 0.002396 0.047278" rpy="0 0 0" />
-    <parent link="base_1" />
-    <child link="forearm_1" />
-    <axis xyz="-0.0 -1.0 -0.0" />
-    <limit upper="-1.57" lower="1.57" effort="100" velocity="100" />
-  </joint>
-  <!--<joint
+  <joint name="HANDCOVER" type="fixed">
+    <origin xyz="-0.00045 -0.0653 0.0842703" rpy="0 0 0" />
+    <parent link="HAND_BASE_PROTO_VER_2_1" />
+    <child link="TOP_COVER_PROTO_VER2_1" />
+  </joint>
+  <!-- finger joints declarations-->
+  <joint name="HAND_pinkybase" type="revolute">
+    <origin xyz="-0.008709 0.0538191 0.14149" rpy="0 0 0" />
+    <parent link="HAND_BASE_PROTO_VER_2_1" />
+    <child link="pinky_finger_base_1" />
+    <axis xyz="-0.0 1.0 -0.0" />
+    <limit upper="1.570796" lower="0.0" effort="100" velocity="100" />
+  </joint>
+  <joint name="pinkybase_pinkymiddle" type="fixed">
+    <origin xyz="0.0 -0.006 0.0485" rpy="0 0 0" />
+    <parent link="pinky_finger_base_1" />
+    <child link="pinky_finger_middle_1" />
+  </joint>
+  <joint name="pinkymiddle_pinkytip" type="fixed">
+    <origin xyz="0.000113 0.0 0.034" rpy="0 0 0" />
+    <parent link="pinky_finger_middle_1" />
+    <child link="pinky_finger_tip_1" />
+  </joint>
+  <joint name="HAND_ringbase" type="revolute">
+    <origin xyz="-0.007035 0.023223 0.157908" rpy="0 0 0" />
+    <parent link="HAND_BASE_PROTO_VER_2_1" />
+    <child link="inder_finger_base_3" />
+    <axis xyz="0.0 1.0 0.0" />
+    <limit upper="0.0" lower="1.570796" effort="100" velocity="100" />
+  </joint>
+  <joint name="ringbase_ringmiddle" type="fixed">
+    <origin xyz="0.0 -0.0 0.062385" rpy="0 0 0" />
+    <parent link="inder_finger_base_3" />
+    <child link="inder_finger_middle_3" />
+  </joint>
+  <joint name="ringmiddle_ringtip" type="fixed">
+    <origin xyz="0.0 0.0 0.038" rpy="0 0 0" />
+    <parent link="inder_finger_middle_3" />
+    <child link="index_finger_tip_3" />
+  </joint>
+  <joint name="HAND_middlebase" type="revolute">
+    <origin xyz="-0.007864 -0.0075 0.161523" rpy="0 0 0" />
+    <parent link="HAND_BASE_PROTO_VER_2_1" />
+    <child link="inder_finger_base_1" />
+    <axis xyz="0.0 -1.0 0.0" />
+    <limit upper="0.0" lower="-1.570796" effort="100" velocity="100" />
+  </joint>
+  <joint name="middlebase_middlemiddle" type="fixed">
+    <origin xyz="0.0 -0.006 0.05" rpy="0 0 0" />
+    <parent link="inder_finger_base_1" />
+    <child link="inder_finger_middle_1" />
+  </joint>
+  <joint name="middlemiddle_middletip" type="fixed">
+    <origin xyz="0.0 0.0 0.038" rpy="0 0 0" />
+    <parent link="inder_finger_middle_1" />
+    <child link="index_finger_tip_1" />
+  </joint>
+  <joint name="HAND_indexbase" type="revolute">
+    <origin xyz="0.000655 -0.0434 0.15487" rpy="0 0 0" />
+    <parent link="HAND_BASE_PROTO_VER_2_1" />
+    <child link="inder_finger_base_2" />
+    <axis xyz="0.0 -1.0 0.0" />
+    <limit upper="0.0" lower="-1.570796" effort="100" velocity="100" />
+  </joint>
+  <joint name="indexbase_indexmiddle" type="fixed">
+    <origin xyz="0.0 -0.0 0.056347" rpy="0 0 0" />
+    <parent link="inder_finger_base_2" />
+    <child link="inder_finger_middle_2" />
+  </joint>
+  <joint name="indexmiddle_indextip" type="fixed">
+    <origin xyz="0.0 0.0 0.032" rpy="0 0 0" />
+    <parent link="inder_finger_middle_2" />
+    <child link="index_finger_tip_2" />
+  </joint>
+  <!-- <joint
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