Commit message: effort controllers working

File: src/robot_description/urdf/BASE_ROBOT_ESSENTIALS.xacro (robot description, xacro)
@@ -1,5 +1,6 @@
 <?xml version="1.0"?>
 <robot xmlns:xacro="http://www.ros.org/wiki/xacro" name="Tayson">
-  <xacro:macro name="base_transmission" params="prefix ">
+  <!--<xacro:macro
+  name="base_transmission" params="prefix ">
     <transmission name="${prefix}_LINK_trans" type="SimpleTransmission">
       <type>transmission_interface/SimpleTransmission</type>
@@ -12,32 +13,72 @@
       </joint>
     </transmission>
-  </xacro:macro>
+</xacro:macro> -->
+  <transmission name="BASE_FOREARM_tran">
+    <type>transmission_interface/SimpleTransmission</type>
+    <joint name="BASE_FOREARM">
+      <hardwareInterface>hardware_interface/EffortJointInterface</hardwareInterface>
+    </joint>
+    <actuator name="BASE_FOREARM_actr">
+      <hardwareInterface>hardware_interface/EffortJointInterface</hardwareInterface>
+      <mechanicalReduction>1</mechanicalReduction>
+    </actuator>
+  </transmission>
   <transmission name="hSERV_HAND_tran">
     <type>transmission_interface/SimpleTransmission</type>
     <joint name="hSERV_HAND">
-      <hardwareInterface>hardware_interface/PositionJointInterface</hardwareInterface>
+      <hardwareInterface>hardware_interface/EffortJointInterface</hardwareInterface>
     </joint>
     <actuator name="hSERV_HAND_actr">
-      <hardwareInterface>hardware_interface/PositionJointInterface</hardwareInterface>
+      <hardwareInterface>hardware_interface/EffortJointInterface</hardwareInterface>
       <mechanicalReduction>1</mechanicalReduction>
     </actuator>
   </transmission>
-  <transmission name="BASE_FOREARM_tran">
+  <transmission name="HAND_pinkybase_tran">
     <type>transmission_interface/SimpleTransmission</type>
-    <joint name="BASE_FOREARM">
-      <hardwareInterface>hardware_interface/PositionJointInterface</hardwareInterface>
+    <joint name="HAND_pinkybase">
+      <hardwareInterface>hardware_interface/EffortJointInterface</hardwareInterface>
     </joint>
-    <actuator name="BASE_FOREARM_actr">
-      <hardwareInterface>hardware_interface/PositionJointInterface</hardwareInterface>
+    <actuator name="HAND_pinkybase_actr">
+      <hardwareInterface>hardware_interface/EffortJointInterface</hardwareInterface>
       <mechanicalReduction>1</mechanicalReduction>
     </actuator>
   </transmission>
-  <transmission name="HAND_thumbbase_tran">
+  <transmission name="HAND_ringbase_tran">
+    <type>transmission_interface/SimpleTransmission</type>
+    <joint name="HAND_ringbase">
+      <hardwareInterface>hardware_interface/EffortJointInterface</hardwareInterface>
+    </joint>
+    <actuator name="HAND_ringbase_actr">
+      <hardwareInterface>hardware_interface/EffortJointInterface</hardwareInterface>
+      <mechanicalReduction>1</mechanicalReduction>
+    </actuator>
+  </transmission>
+  <transmission name="HAND_middlebase_tran">
+    <type>transmission_interface/SimpleTransmission</type>
+    <joint name="HAND_middlebase">
+      <hardwareInterface>hardware_interface/EffortJointInterface</hardwareInterface>
+    </joint>
+    <actuator name="HAND_middlebase_actr">
+      <hardwareInterface>hardware_interface/EffortJointInterface</hardwareInterface>
+      <mechanicalReduction>1</mechanicalReduction>
+    </actuator>
+  </transmission>
+  <transmission name="HAND_indexbase_tran">
+    <type>transmission_interface/SimpleTransmission</type>
+    <joint name="HAND_indexbase">
+      <hardwareInterface>hardware_interface/EffortJointInterface</hardwareInterface>
+    </joint>
+    <actuator name="HAND_indexbase_actr">
+      <hardwareInterface>hardware_interface/EffortJointInterface</hardwareInterface>
+      <mechanicalReduction>1</mechanicalReduction>
+    </actuator>
+  </transmission>
+  <!-- <transmission name="HAND_thumbbase_tran">
     <type>transmission_interface/SimpleTransmission</type>
     <joint name="HAND_thumbbase">
-      <hardwareInterface>hardware_interface/PositionJointInterface</hardwareInterface>
+      <hardwareInterface>hardware_interface/EffortJointInterface</hardwareInterface>
     </joint>
     <actuator name="HAND_thumbbase_actr">
-      <hardwareInterface>hardware_interface/PositionJointInterface</hardwareInterface>
+      <hardwareInterface>hardware_interface/EffortJointInterface</hardwareInterface>
       <mechanicalReduction>1</mechanicalReduction>
     </actuator>
@@ -46,8 +87,8 @@
     <type>transmission_interface/SimpleTransmission</type>
     <joint name="thumbbase_thumbmiddle">
-      <hardwareInterface>hardware_interface/PositionJointInterface</hardwareInterface>
+      <hardwareInterface>hardware_interface/EffortJointInterface</hardwareInterface>
     </joint>
     <actuator name="thumbbase_thumbmiddle_actr">
-      <hardwareInterface>hardware_interface/PositionJointInterface</hardwareInterface>
+      <hardwareInterface>hardware_interface/EffortJointInterface</hardwareInterface>
       <mechanicalReduction>1</mechanicalReduction>
     </actuator>
@@ -56,18 +97,8 @@
     <type>transmission_interface/SimpleTransmission</type>
     <joint name="thumbmiddle_thumbtip">
-      <hardwareInterface>hardware_interface/PositionJointInterface</hardwareInterface>
+      <hardwareInterface>hardware_interface/EffortJointInterface</hardwareInterface>
     </joint>
     <actuator name="thumbmiddle_thumbtip_actr">
-      <hardwareInterface>hardware_interface/PositionJointInterface</hardwareInterface>
-      <mechanicalReduction>1</mechanicalReduction>
-    </actuator>
-  </transmission>
-  <transmission name="HAND_pinkybase_tran">
-    <type>transmission_interface/SimpleTransmission</type>
-    <joint name="HAND_pinkybase">
-      <hardwareInterface>hardware_interface/PositionJointInterface</hardwareInterface>
-    </joint>
-    <actuator name="HAND_pinkybase_actr">
-      <hardwareInterface>hardware_interface/PositionJointInterface</hardwareInterface>
+      <hardwareInterface>hardware_interface/EffortJointInterface</hardwareInterface>
       <mechanicalReduction>1</mechanicalReduction>
     </actuator>
@@ -76,8 +107,8 @@
     <type>transmission_interface/SimpleTransmission</type>
     <joint name="pinkybase_pinkymiddle">
-      <hardwareInterface>hardware_interface/PositionJointInterface</hardwareInterface>
+      <hardwareInterface>hardware_interface/EffortJointInterface</hardwareInterface>
     </joint>
     <actuator name="pinkybase_pinkymiddle_actr">
-      <hardwareInterface>hardware_interface/PositionJointInterface</hardwareInterface>
+      <hardwareInterface>hardware_interface/EffortJointInterface</hardwareInterface>
       <mechanicalReduction>1</mechanicalReduction>
     </actuator>
@@ -86,18 +117,8 @@
     <type>transmission_interface/SimpleTransmission</type>
     <joint name="pinkymiddle_pinkytip">
-      <hardwareInterface>hardware_interface/PositionJointInterface</hardwareInterface>
+      <hardwareInterface>hardware_interface/EffortJointInterface</hardwareInterface>
     </joint>
     <actuator name="pinkymiddle_pinkytip_actr">
-      <hardwareInterface>hardware_interface/PositionJointInterface</hardwareInterface>
-      <mechanicalReduction>1</mechanicalReduction>
-    </actuator>
-  </transmission>
-  <transmission name="HAND_ringbase_tran">
-    <type>transmission_interface/SimpleTransmission</type>
-    <joint name="HAND_ringbase">
-      <hardwareInterface>hardware_interface/PositionJointInterface</hardwareInterface>
-    </joint>
-    <actuator name="HAND_ringbase_actr">
-      <hardwareInterface>hardware_interface/PositionJointInterface</hardwareInterface>
+      <hardwareInterface>hardware_interface/EffortJointInterface</hardwareInterface>
       <mechanicalReduction>1</mechanicalReduction>
     </actuator>
@@ -106,8 +127,8 @@
     <type>transmission_interface/SimpleTransmission</type>
     <joint name="ringbase_ringmiddle">
-      <hardwareInterface>hardware_interface/PositionJointInterface</hardwareInterface>
+      <hardwareInterface>hardware_interface/EffortJointInterface</hardwareInterface>
     </joint>
     <actuator name="ringbase_ringmiddle_actr">
-      <hardwareInterface>hardware_interface/PositionJointInterface</hardwareInterface>
+      <hardwareInterface>hardware_interface/EffortJointInterface</hardwareInterface>
       <mechanicalReduction>1</mechanicalReduction>
     </actuator>
@@ -116,18 +137,8 @@
     <type>transmission_interface/SimpleTransmission</type>
     <joint name="ringmiddle_ringtip">
-      <hardwareInterface>hardware_interface/PositionJointInterface</hardwareInterface>
+      <hardwareInterface>hardware_interface/EffortJointInterface</hardwareInterface>
     </joint>
     <actuator name="ringmiddle_ringtip_actr">
-      <hardwareInterface>hardware_interface/PositionJointInterface</hardwareInterface>
-      <mechanicalReduction>1</mechanicalReduction>
-    </actuator>
-  </transmission>
-  <transmission name="HAND_middlebase_tran">
-    <type>transmission_interface/SimpleTransmission</type>
-    <joint name="HAND_middlebase">
-      <hardwareInterface>hardware_interface/PositionJointInterface</hardwareInterface>
-    </joint>
-    <actuator name="HAND_middlebase_actr">
-      <hardwareInterface>hardware_interface/PositionJointInterface</hardwareInterface>
+      <hardwareInterface>hardware_interface/EffortJointInterface</hardwareInterface>
       <mechanicalReduction>1</mechanicalReduction>
     </actuator>
@@ -136,8 +147,8 @@
     <type>transmission_interface/SimpleTransmission</type>
     <joint name="middlebase_middlemiddle">
-      <hardwareInterface>hardware_interface/PositionJointInterface</hardwareInterface>
+      <hardwareInterface>hardware_interface/EffortJointInterface</hardwareInterface>
     </joint>
     <actuator name="middlebase_middlemiddle_actr">
-      <hardwareInterface>hardware_interface/PositionJointInterface</hardwareInterface>
+      <hardwareInterface>hardware_interface/EffortJointInterface</hardwareInterface>
       <mechanicalReduction>1</mechanicalReduction>
     </actuator>
@@ -146,18 +157,8 @@
     <type>transmission_interface/SimpleTransmission</type>
     <joint name="middlemiddle_middletip">
-      <hardwareInterface>hardware_interface/PositionJointInterface</hardwareInterface>
+      <hardwareInterface>hardware_interface/EffortJointInterface</hardwareInterface>
     </joint>
     <actuator name="middlemiddle_middletip_actr">
-      <hardwareInterface>hardware_interface/PositionJointInterface</hardwareInterface>
-      <mechanicalReduction>1</mechanicalReduction>
-    </actuator>
-  </transmission>
-  <transmission name="HAND_indexbase_tran">
-    <type>transmission_interface/SimpleTransmission</type>
-    <joint name="HAND_indexbase">
-      <hardwareInterface>hardware_interface/PositionJointInterface</hardwareInterface>
-    </joint>
-    <actuator name="HAND_indexbase_actr">
-      <hardwareInterface>hardware_interface/PositionJointInterface</hardwareInterface>
+      <hardwareInterface>hardware_interface/EffortJointInterface</hardwareInterface>
       <mechanicalReduction>1</mechanicalReduction>
     </actuator>
@@ -166,8 +167,8 @@
     <type>transmission_interface/SimpleTransmission</type>
     <joint name="indexbase_indexmiddle">
-      <hardwareInterface>hardware_interface/PositionJointInterface</hardwareInterface>
+      <hardwareInterface>hardware_interface/EffortJointInterface</hardwareInterface>
     </joint>
     <actuator name="indexbase_indexmiddle_actr">
-      <hardwareInterface>hardware_interface/PositionJointInterface</hardwareInterface>
+      <hardwareInterface>hardware_interface/EffortJointInterface</hardwareInterface>
       <mechanicalReduction>1</mechanicalReduction>
     </actuator>
@@ -176,10 +177,10 @@
     <type>transmission_interface/SimpleTransmission</type>
     <joint name="indexmiddle_indextip">
-      <hardwareInterface>hardware_interface/PositionJointInterface</hardwareInterface>
+      <hardwareInterface>hardware_interface/EffortJointInterface</hardwareInterface>
     </joint>
     <actuator name="indexmiddle_indextip_actr">
-      <hardwareInterface>hardware_interface/PositionJointInterface</hardwareInterface>
+      <hardwareInterface>hardware_interface/EffortJointInterface</hardwareInterface>
       <mechanicalReduction>1</mechanicalReduction>
     </actuator>
-  </transmission>
+  </transmission> -->
 </robot>

Commit message: ubuntu issues

File: src/robot_description/urdf/BASE_ROBOT.urdf.xacro (robot description, xacro)
@@ -606,5 +606,5 @@
     </collision>
   </link>
-  <joint name="RFW_JOINT" type="continuous">
+  <joint name="RFW_JOINT" type="fixed">
     <origin xyz="0.1 -0.1 0.03145" rpy="0 0 0" />
     <parent link="base_link" />
@@ -612,5 +612,5 @@
     <axis xyz="-0.0 -1.0 -0.0" />
   </joint>
-  <joint name="RBW_JOINT" type="continuous">
+  <joint name="RBW_JOINT" type="fixed">
     <origin xyz="-0.1 -0.1 0.03145" rpy="0 0 0" />
     <parent link="base_link" />
@@ -618,5 +618,5 @@
     <axis xyz="-0.0 -1.0 -0.0" />
   </joint>
-  <joint name="LFW_JOINT" type="continuous">
+  <joint name="LFW_JOINT" type="fixed">
     <origin xyz="0.1 0.1 0.03145" rpy="0 0 0" />
     <parent link="base_link" />
@@ -624,5 +624,5 @@
     <axis xyz="0.0 1.0 0.0" />
   </joint>
-  <joint name="LBW_JOINT" type="continuous">
+  <joint name="LBW_JOINT" type="fixed">
     <origin xyz="-0.1 0.1 0.03145" rpy="0 0 0" />
     <parent link="base_link" />
@@ -650,5 +650,5 @@
     <child link="forearm_1" />
     <axis xyz="-0.0 -1.0 -0.0" />
-    <limit upper="1.57" lower="-1.57" effort="50" velocity="-1" />
+    <limit upper="1.40" lower="-1.40" effort="50" velocity="-1" />
   </joint>
   <joint name="FOREARM_hSERV" type="fixed">
@@ -662,5 +662,5 @@
     <child link="HAND_BASE_PROTO_VER_2_1" />
     <axis xyz="0.0 -0.0 -1.0" />
-    <limit upper="1.570796" lower="-1.57" effort="100" velocity="100" />
+    <limit upper="1.570796" lower="-1.57" effort="50" velocity="10" />
   </joint>
   <joint name="HANDCOVER" type="fixed">
@@ -675,5 +675,5 @@
     <child link="pinky_finger_base_1" />
     <axis xyz="-0.0 1.0 -0.0" />
-    <limit upper="1.570796" lower="0.0" effort="100" velocity="100" />
+    <limit upper="1.570796" lower="0.0" effort="50" velocity="10" />
   </joint>
   <joint name="pinkybase_pinkymiddle" type="fixed">
@@ -692,5 +692,5 @@
     <child link="inder_finger_base_3" />
     <axis xyz="0.0 1.0 0.0" />
-    <limit upper="0.0" lower="1.570796" effort="100" velocity="100" />
+    <limit upper="1.570796" lower="0.0" effort="10" velocity="10" />
   </joint>
   <joint name="ringbase_ringmiddle" type="fixed">
@@ -709,5 +709,5 @@
     <child link="inder_finger_base_1" />
     <axis xyz="0.0 -1.0 0.0" />
-    <limit upper="0.0" lower="-1.570796" effort="100" velocity="100" />
+    <limit upper="0.0" lower="-1.570796" effort="10" velocity="10" />
   </joint>
   <joint name="middlebase_middlemiddle" type="fixed">
@@ -726,5 +726,5 @@
     <child link="inder_finger_base_2" />
     <axis xyz="0.0 -1.0 0.0" />
-    <limit upper="0.0" lower="-1.570796" effort="100" velocity="100" />
+    <limit upper="0.0" lower="-1.570796" effort="10" velocity="10" />
   </joint>
   <joint name="indexbase_indexmiddle" type="fixed">
@@ -743,20 +743,16 @@
   <parent link="HAND_BASE_PROTO_VER_2_1"/>
   <child link="pinky_finger_base_2"/>
-  <axis xyz="-0 0 1"/>
+  <axis xyz="0 1 0"/>
   <limit upper="3.839724" lower="3.141593" effort="100" velocity="100"/>
 </joint>
-<joint name="thumbbase_thumbmiddle" type="revolute">
+<joint name="thumbbase_thumbmiddle" type="fixed">
   <origin xyz="0.075734 -0.311296 -0.155475" rpy="0 0 0"/>
   <parent link="pinky_finger_base_2"/>
   <child link="pinky_finger_middle_2"/>
-  <axis xyz="0.694658 -0.095071 -0.71303"/>
-  <limit upper="0.0" lower="-1.570796" effort="100" velocity="100"/>
 </joint>
-<joint name="thumbmiddle_thumbtip" type="revolute">
+<joint name="thumbmiddle_thumbtip" type="fixed">
   <origin xyz="0.000113 -0.006 0.034" rpy="0 0 0"/>
   <parent link="pinky_finger_middle_2"/>
   <child link="pinky_finger_tip_2"/>
-  <axis xyz="0.694658 -0.095071 -0.71303"/>
-  <limit upper="0.0" lower="-0.436332" effort="100" velocity="100"/>
 </joint> -->
 </robot>

File: src/robot_description/urdf/BASE_ROBOT_ESSENTIALS.xacro (robot description, xacro)
@@ -74,5 +74,5 @@
     </actuator>
   </transmission>
-  <!-- <transmission name="HAND_thumbbase_tran">
+   <!-- <transmission name="HAND_thumbbase_tran">
     <type>transmission_interface/SimpleTransmission</type>
     <joint name="HAND_thumbbase">
@@ -83,6 +83,6 @@
       <mechanicalReduction>1</mechanicalReduction>
     </actuator>
-  </transmission>
-  <transmission name="thumbbase_thumbmiddle_tran">
+  </transmission> -->
+  <!--<transmission name="thumbbase_thumbmiddle_tran">
     <type>transmission_interface/SimpleTransmission</type>
     <joint name="thumbbase_thumbmiddle">
@@ -103,6 +103,6 @@
       <mechanicalReduction>1</mechanicalReduction>
     </actuator>
-  </transmission>
-  <transmission name="pinkybase_pinkymiddle_tran">
+  </transmission> -->
+  <!-- <transmission name="pinkybase_pinkymiddle_tran">
     <type>transmission_interface/SimpleTransmission</type>
     <joint name="pinkybase_pinkymiddle">

Commit message: Reverted to rosserial for base communication

File: src/robot_description/urdf/BASE_ROBOT.urdf.xacro (robot description, xacro)
@@ -631,5 +631,5 @@
   </joint>
   <joint name="BASE_mBASE" type="fixed">
-    <origin xyz="0.15 0.0 0.014" rpy="0 0 0" />
+    <origin xyz="0.05 0.0 0.014" rpy="0 0 0" />
     <parent link="base_link" />
     <child link="base_1" />
@@ -650,5 +650,5 @@
     <child link="forearm_1" />
     <axis xyz="-0.0 -1.0 -0.0" />
-    <limit upper="1.40" lower="-1.40" effort="50" velocity="-1" />
+    <limit upper="1.40" lower="-1.40" effort="26" velocity="-1" />
   </joint>
   <joint name="FOREARM_hSERV" type="fixed">
@@ -662,5 +662,5 @@
     <child link="HAND_BASE_PROTO_VER_2_1" />
     <axis xyz="0.0 -0.0 -1.0" />
-    <limit upper="1.570796" lower="-1.57" effort="50" velocity="10" />
+    <limit upper="1.570796" lower="-1.57" effort="13" velocity="10" />
   </joint>
   <joint name="HANDCOVER" type="fixed">
@@ -675,5 +675,5 @@
     <child link="pinky_finger_base_1" />
     <axis xyz="-0.0 1.0 -0.0" />
-    <limit upper="1.570796" lower="0.0" effort="50" velocity="10" />
+    <limit upper="1.570796" lower="0.0" effort="7" velocity="10" />
   </joint>
   <joint name="pinkybase_pinkymiddle" type="fixed">
@@ -692,5 +692,5 @@
     <child link="inder_finger_base_3" />
     <axis xyz="0.0 1.0 0.0" />
-    <limit upper="1.570796" lower="0.0" effort="10" velocity="10" />
+    <limit upper="1.570796" lower="0.0" effort="7" velocity="10" />
   </joint>
   <joint name="ringbase_ringmiddle" type="fixed">
@@ -709,5 +709,5 @@
     <child link="inder_finger_base_1" />
     <axis xyz="0.0 -1.0 0.0" />
-    <limit upper="0.0" lower="-1.570796" effort="10" velocity="10" />
+    <limit upper="0.0" lower="-1.570796" effort="7" velocity="10" />
   </joint>
   <joint name="middlebase_middlemiddle" type="fixed">
@@ -726,5 +726,5 @@
     <child link="inder_finger_base_2" />
     <axis xyz="0.0 -1.0 0.0" />
-    <limit upper="0.0" lower="-1.570796" effort="10" velocity="10" />
+    <limit upper="0.0" lower="-1.570796" effort="7" velocity="10" />
   </joint>
   <joint name="indexbase_indexmiddle" type="fixed">

Commit message: removed trial files and updated servo control

File: src/robot_description/urdf/BASE_ROBOT.urdf.xacro (robot description, xacro)
@@ -650,5 +650,5 @@
     <child link="forearm_1" />
     <axis xyz="-0.0 -1.0 -0.0" />
-    <limit upper="1.40" lower="-1.40" effort="26" velocity="-1" />
+    <limit upper="0.45" lower="-1.40" effort="26" velocity="-1" />
   </joint>
   <joint name="FOREARM_hSERV" type="fixed">
